File: ProjectCARS/ProjectCARS.kicad_sch (KiCad schematic)
At the start: 0 parts

Commit message: Rover Schematic
Parts:
- added 7.4V: Battery, symbol Device:Battery
- added A?: Motor Control Shield, Module:Arduino_UNO_R3, symbol Custom Parts:Motor_Control_Shield
- added C1: 100uF, symbol Device:C_Polarized
- added M1, M2, M3, M4: Motor_DC, symbol Motor:Motor_DC
- added R1: 1k, symbol Device:R
- added R2: 2k, symbol Device:R
- added U: ESP32 S3 Dev Module, symbol Custom Parts:_1
Connections:
- new net: A?.16 (M3+), M3.1 (+)
- new net: A?.15 (M3-), M3.2 (-)
- new net: A?.7 (A1), R1.1, R2.1
- new net: R1.2, U.23 (GPIO17)
- new net: A?.17 (M2+), M2.1 (+)
- new net: A?.18 (M2-), M2.2 (-)
- new net: A?.1 (+5V), C1.1, U.55 (VDDA), U.56 (VDDA)
- new net: A?.12 (M4-), M4.2 (-)
- new net: A?.13 (M4+), M4.1 (+)
- new net: A?.20 (M1-), M1.2 (-)
- new net: A?.21 (M1+), M1.1 (+)
- new net: 7.4V.1 (+), A?.4 (Ext_PWR+)
- new net: A?.6 (A0), U.19 (GPIO16)
- new net: U.2 (VDD3P3), U.3 (VDD3P3)
- new net GND: 7.4V.2 (-), A?.3 (Ext_PWR-), A?.5 (GND), C1.2, R2.2, U.57 (GND)

Commit message: New Schematics/Clean Up Comments
Parts:
- added MPU6500: ~, symbol Custom Parts:MPU6500
- added SW? (x2): SW_Push, symbol Switch:SW_Push
- added U?: DOIT SP32 DEVKIT V1, symbol Custom Parts:_1
Connections:
- net GND: now also MPU6500.2 (GND), U?.57 (GND)
- net at A?.1 (+5V): now also C1.1, U.55 (VDDA), U.56 (VDDA)
- new net: MPU6500.1 (VCC), U?.2 (VDD3P3), U?.3 (VDD3P3)
- new net +5V: U?.55 (VDDA), U?.56 (VDDA)
